File: Pcb/esp_radio/io_expander.kicad_sch (KiCad schematic)
At the start: 17 parts, among them J9 GPIO, SW3 Next, SW4 RotaryEncoder_Switch, SW5 Play, SW6 Prev, U9 MCP23017_SO

Commit message: Move custom components to kicad_common_library.
Parts:
- added J5: GPIOB, symbol Connector_Generic:Conn_01x03
- J6: renamed from J9; value GPIO -> GPIOA
- renumbered SW6 to SW3, SW5 to SW4, SW3 to SW5, SW4 to SW6, U9 to U7
Connections:
- net at U7.6 (GPB5): now also J5.1 (Pin_1)
- net at U7.7 (GPB6): now also J5.2 (Pin_2)
- net at U7.8 (GPB7): now also J5.3 (Pin_3)
Changed lines of the file:
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@@
+    (stroke (width 0) (type default))
+  )
+  (wire (pts (xy 140.97 62.23) (xy 144.78 62.23))
     (stroke (width 0) (type default))
   )
@@
     (stroke (width 0) (type default))
   )
+  (wire (pts (xy 140.97 59.69) (xy 144.78 59.69))
+    (stroke (width 0) (type default))
+  )
   (wire (pts (xy 250.19 35.56) (xy 250.19 30.48))
     (stroke (width 0) (type default))
@@
   )
   (wire (pts (xy 226.06 74.93) (xy 226.06 80.01))
+    (stroke (width 0) (type default))
+  )
+  (wire (pts (xy 140.97 64.77) (xy 144.78 64.77))
     (stroke (width 0) (type default))
   )
@@
   (symbol (lib_id "Device:RotaryEncoder_Switch") (at 260.35 113.03 0) (unit 1)
     (in_bom yes) (on_board yes) (dnp no) (fields_autoplaced)
-    (property "Reference" "SW4" (at 260.35 104.14 0)
+    (property "Reference" "SW6" (at 260.35 104.14 0)
       (effects (font (size 1.27 1.27)))
     )
@@
       (project "esp_radio"
         (path "/c9e2e0d2-0655-4f5e-8e13-71b41b1f7cfe/6c8b235f-e3ea-4277-bdf9-de9910b169f3"
-          (reference "SW4") (unit 1)
+          (reference "SW6") (unit 1)
         )
       )
@@
   (symbol (lib_id "power:GND") (at 123.19 100.33 0) (unit 1)
     (in_bom yes) (on_board yes) (dnp no) (fields_autoplaced)
-    (property "Reference" "#PWR053" (at 123.19 106.68 0)
+    (property "Reference" "#PWR046" (at 123.19 106.68 0)
       (effects (font (size 1.27 1.27)) hide)
     )
@@
       (project "esp_radio"
         (path "/c9e2e0d2-0655-4f5e-8e13-71b41b1f7cfe/6c8b235f-e3ea-4277-bdf9-de9910b169f3"
-          (reference "#PWR053") (unit 1)
+          (reference "#PWR046") (unit 1)
         )
       )
@@
         )
         (path "/c9e2e0d2-0655-4f5e-8e13-71b41b1f7cfe/6c8b235f-e3ea-4277-bdf9-de9910b169f3"
-          (reference "C39") (unit 1)
+          (reference "C37") (unit 1)
         )
       )
@@
         )
         (path "/c9e2e0d2-0655-4f5e-8e13-71b41b1f7cfe/6c8b235f-e3ea-4277-bdf9-de9910b169f3"
-          (reference "R26") (unit 1)
+          (reference "R23") (unit 1)
         )
       )
@@
   (symbol (lib_id "Switch:SW_Push_Dual") (at 260.35 54.61 0) (unit 1)
     (in_bom yes) (on_board yes) (dnp no) (fields_autoplaced)
-    (property "Reference" "SW5" (at 260.35 48.26 0)
+    (property "Reference" "SW4" (at 260.35 48.26 0)
       (effects (font (size 1.27 1.27)))
     )
@@
       (project "esp_radio"
         (path "/c9e2e0d2-0655-4f5e-8e13-71b41b1f7cfe/6c8b235f-e3ea-4277-bdf9-de9910b169f3"
-          (reference "SW5") (unit 1)
+          (reference "SW4") (unit 1)
         )
       )
@@
         )
         (path "/c9e2e0d2-0655-4f5e-8e13-71b41b1f7cfe/6c8b235f-e3ea-4277-bdf9-de9910b169f3"
-          (reference "C40") (unit 1)
+          (reference "C38") (unit 1)
         )
       )
@@
         )
         (path "/c9e2e0d2-0655-4f5e-8e13-71b41b1f7cfe/6c8b235f-e3ea-4277-bdf9-de9910b169f3"
-          (reference "C37") (unit 1)
+          (reference "C35") (unit 1)
         )
       )
@@
   (symbol (lib_id "power:GND") (at 278.13 137.16 0) (unit 1)
     (in_bom yes) (on_board yes) (dnp no) (fields_autoplaced)
-    (property "Reference" "#PWR051" (at 278.13 143.51 0)
+    (property "Reference" "#PWR047" (at 278.13 143.51 0)
       (effects (font (size 1.27 1.27)) hide)
     )
@@
       (project "esp_radio"
         (path "/c9e2e0d2-0655-4f5e-8e13-71b41b1f7cfe/6c8b235f-e3ea-4277-bdf9-de9910b169f3"
-          (reference "#PWR051") (unit 1)
+          (reference "#PWR047") (unit 1)
         )
       )
@@
         )
         (path "/c9e2e0d2-0655-4f5e-8e13-71b41b1f7cfe/6c8b235f-e3ea-4277-bdf9-de9910b169f3"
-          (reference "#PWR054") (unit 1)
+          (reference "#PWR043") (unit 1)
         )
       )
@@
   (symbol (lib_id "Interface_Expansion:MCP23017_SO") (at 123.19 67.31 0) (unit 1)
     (in_bom yes) (on_board yes) (dnp no) (fields_autoplaced)
-    (property "Reference" "U9" (at 125.1459 40.64 0)
+    (property "Reference" "U7" (at 125.1459 40.64 0)
       (effects (font (size 1.27 1.27)) (justify left))
     )
@@
       (project "esp_radio"
         (path "/c9e2e0d2-0655-4f5e-8e13-71b41b1f7cfe/6c8b235f-e3ea-4277-bdf9-de9910b169f3"
-          (reference "U9") (unit 1)
+          (reference "U7") (unit 1)
         )
       )
@@
   (symbol (lib_id "Connector_Generic:Conn_01x02") (at 152.4 85.09 0) (unit 1)
     (in_bom yes) (on_board yes) (dnp no) (fields_autoplaced)
-    (property "Reference" "J9" (at 154.94 85.725 0)
+    (property "Reference" "J6" (at 154.94 85.725 0)
       (effects (font (size 1.27 1.27)) (justify left))
     )
-    (property "Value" "GPIO" (at 154.94 88.265 0)
+    (property "Value" "GPIOA" (at 154.94 88.265 0)
       (effects (font (size 1.27 1.27)) (justify left))
     )
@@
       (project "esp_radio"
         (path "/c9e2e0d2-0655-4f5e-8e13-71b41b1f7cfe/6c8b235f-e3ea-4277-bdf9-de9910b169f3"
-          (reference "J9") (unit 1)
+          (reference "J6") (unit 1)
         )
       )
@@
   (symbol (lib_id "power:GND") (at 248.92 143.51 0) (unit 1)
     (in_bom yes) (on_board yes) (dnp no) (fields_autoplaced)
-    (property "Reference" "#PWR052" (at 248.92 149.86 0)
+    (property "Reference" "#PWR048" (at 248.92 149.86 0)
       (effects (font (size 1.27 1.27)) hide)
     )
@@
       (project "esp_radio"
         (path "/c9e2e0d2-0655-4f5e-8e13-71b41b1f7cfe/6c8b235f-e3ea-4277-bdf9-de9910b169f3"
-          (reference "#PWR052") (unit 1)
+          (reference "#PWR048") (unit 1)
         )
       )
@@
         )
         (path "/c9e2e0d2-0655-4f5e-8e13-71b41b1f7cfe/6c8b235f-e3ea-4277-bdf9-de9910b169f3"
-          (reference "C36") (unit 1)
+          (reference "C34") (unit 1)
         )
       )
@@
         )
         (path "/c9e2e0d2-0655-4f5e-8e13-71b41b1f7cfe/6c8b235f-e3ea-4277-bdf9-de9910b169f3"
-          (reference "R25") (unit 1)
+          (reference "R26") (unit 1)
         )
       )
@@
         )
         (path "/c9e2e0d2-0655-4f5e-8e13-71b41b1f7cfe/6c8b235f-e3ea-4277-bdf9-de9910b169f3"
-          (reference "C41") (unit 1)
+          (reference "C39") (unit 1)
         )
       )
@@
   (symbol (lib_id "Switch:SW_Push_Dual") (at 260.35 30.48 0) (unit 1)
     (in_bom yes) (on_board yes) (dnp no) (fields_autoplaced)
-    (property "Reference" "SW6" (at 260.35 24.13 0)
+    (property "Reference" "SW3" (at 260.35 24.13 0)
       (effects (font (size 1.27 1.27)))
     )
@@
       (project "esp_radio"
         (path "/c9e2e0d2-0655-4f5e-8e13-71b41b1f7cfe/6c8b235f-e3ea-4277-bdf9-de9910b169f3"
-          (reference "SW6") (unit 1)
+          (reference "SW3") (unit 1)
         )
       )
@@
         )
         (path "/c9e2e0d2-0655-4f5e-8e13-71b41b1f7cfe/6c8b235f-e3ea-4277-bdf9-de9910b169f3"
-          (reference "C42") (unit 1)
+          (reference "C40") (unit 1)
         )
       )
@@
         )
         (path "/c9e2e0d2-0655-4f5e-8e13-71b41b1f7cfe/6c8b235f-e3ea-4277-bdf9-de9910b169f3"
-          (reference "#PWR055") (unit 1)
+          (reference "#PWR045") (unit 1)
         )
       )
@@
         )
         (path "/c9e2e0d2-0655-4f5e-8e13-71b41b1f7cfe/6c8b235f-e3ea-4277-bdf9-de9910b169f3"
-          (reference "R24") (unit 1)
+          (reference "R25") (unit 1)
         )
       )
@@
         )
         (path "/c9e2e0d2-0655-4f5e-8e13-71b41b1f7cfe/6c8b235f-e3ea-4277-bdf9-de9910b169f3"
-          (reference "R23") (unit 1)
+          (reference "R24") (unit 1)
         )
       )
@@
   (symbol (lib_id "Switch:SW_Push_Dual") (at 260.35 80.01 0) (unit 1)
     (in_bom yes) (on_board yes) (dnp no) (fields_autoplaced)
-    (property "Reference" "SW3" (at 260.35 73.66 0)
+    (property "Reference" "SW5" (at 260.35 73.66 0)
       (effects (font (size 1.27 1.27)))
     )
@@
       (project "esp_radio"
         (path "/c9e2e0d2-0655-4f5e-8e13-71b41b1f7cfe/6c8b235f-e3ea-4277-bdf9-de9910b169f3"
-          (reference "SW3") (unit 1)
+          (reference "SW5") (unit 1)
         )
       )
@@
   (symbol (lib_id "power:GND") (at 100.33 30.48 270) (unit 1)
     (in_bom yes) (on_board yes) (dnp no) (fields_autoplaced)
-    (property "Reference" "#PWR056" (at 93.98 30.48 0)
+    (property "Reference" "#PWR044" (at 93.98 30.48 0)
       (effects (font (size 1.27 1.27)) hide)
     )
@@
       (project "esp_radio"
         (path "/c9e2e0d2-0655-4f5e-8e13-71b41b1f7cfe/6c8b235f-e3ea-4277-bdf9-de9910b169f3"
-          (reference "#PWR056") (unit 1)
+          (reference "#PWR044") (unit 1)
+        )
+      )
+    )
+  )
+  (symbol (lib_id "Connector_Generic:Conn_01x03") (at 149.86 62.23 0) (unit 1)
+    (in_bom yes) (on_board yes) (dnp no) (fields_autoplaced)
+    (property "Reference" "J5" (at 152.4 61.595 0)
+      (effects (font (size 1.27 1.27)) (justify left))
+    )
+    (property "Value" "GPIOB" (at 152.4 64.135 0)
+      (effects (font (size 1.27 1.27)) (justify left))
+    )
+    (property "Footprint" "" (at 149.86 62.23 0)
+      (effects (font (size 1.27 1.27)) hide)
+    )
+    (property "Datasheet" "~" (at 149.86 62.23 0)
+      (effects (font (size 1.27 1.27)) hide)
+    )
+    (pin "1")
+    (pin "2")
+    (pin "3")
+    (instances
+      (project "esp_radio"
+        (path "/c9e2e0d2-0655-4f5e-8e13-71b41b1f7cfe/6c8b235f-e3ea-4277-bdf9-de9910b169f3"
+          (reference "J5") (unit 1)
         )
       )
@@
         )
         (path "/c9e2e0d2-0655-4f5e-8e13-71b41b1f7cfe/6c8b235f-e3ea-4277-bdf9-de9910b169f3"
-          (reference "C38") (unit 1)
-        )
-      )
+          (reference "C36") (unit 1)
+        )
+      )

Commit message: Add components layout on PCB
Parts:
- C24: footprint (none) -> kicad_common_lib:C_0805
- J5: footprint (none) -> Connector_PinHeader_2.54mm:PinHeader_1x03_P2.54mm_Vertical
- J6: footprint (none) -> Connector_PinHeader_2.54mm:PinHeader_1x02_P2.54mm_Vertical
- R19: footprint (none) -> kicad_common_lib:R_0805
- SW3, SW4, SW5: footprint (none) -> kicad_common_lib:SW_PUSH_6mm_H12mm; symbol Switch:SW_Push_Dual -> Switch:SW_Push
- SW6: footprint (none) -> kicad_common_lib:RotaryEncoder_EC16-Switch_Vertical_H20mm
Connections:
- net GND: no longer SW3.4, SW4.4, SW5.4
- net at C24.2, SW5.1, U7.23 (GPA2): no longer SW5.3
- net at C24.2, SW4.1, U7.22 (GPA1): no longer SW4.3
- net at C24.2, SW3.1, U7.21 (GPA0): no longer SW3.3
- net ~{LCD_POWER} renamed LCD_POWER
Other:
- moved on the sheet: C24

Commit message: Add chip select emulation for i2c devices
Parts:
- removed J5: GPIOB, Connector_PinHeader_2.54mm:PinHeader_1x03_P2.54mm_Vertical, symbol Connector_Generic:Conn_01x03
- added J5: GPIOB, Connector_PinHeader_2.54mm:PinHeader_1x01_P2.54mm_Vertical, symbol Connector_Generic:Conn_01x01
Connections:
- net MerusChipSelect: now reaches U7.6 (GPB5)
- net RadioChipSelect: now reaches U7.7 (GPB6)
- net at U7.8 (GPB7): now also J5.1 (Pin_1)
Changed lines of the file:
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@@
     (stroke (width 0) (type default))
   )
-  (wire (pts (xy 140.97 62.23) (xy 144.78 62.23))
+  (wire (pts (xy 140.97 62.23) (xy 158.75 62.23))
     (stroke (width 0) (type default))
   )
@@
     (stroke (width 0) (type default))
   )
-  (wire (pts (xy 140.97 59.69) (xy 144.78 59.69))
+  (wire (pts (xy 140.97 59.69) (xy 161.29 59.69))
     (stroke (width 0) (type default))
   )
@@
     (stroke (width 0) (type default))
   )
+  (wire (pts (xy 158.75 67.31) (xy 176.53 67.31))
+    (stroke (width 0) (type default))
+  )
   (wire (pts (xy 256.54 63.5) (xy 250.19 63.5))
     (stroke (width 0) (type default))
@@
     (stroke (width 0) (type default))
   )
+  (wire (pts (xy 161.29 64.77) (xy 176.53 64.77))
+    (stroke (width 0) (type default))
+  )
   (wire (pts (xy 140.97 72.39) (xy 238.76 72.39))
     (stroke (width 0) (type default))
@@
     (stroke (width 0) (type default))
   )
+  (wire (pts (xy 158.75 62.23) (xy 158.75 67.31))
+    (stroke (width 0) (type default))
+  )
   (wire (pts (xy 101.6 69.85) (xy 105.41 69.85))
     (stroke (width 0) (type default))
@@
   )
   (wire (pts (xy 140.97 74.93) (xy 226.06 74.93))
+    (stroke (width 0) (type default))
+  )
+  (wire (pts (xy 161.29 59.69) (xy 161.29 64.77))
     (stroke (width 0) (type default))
   )
@@
     (effects (font (size 1.27 1.27)) (justify left))
   )
+  (hierarchical_label "RadioChipSelect" (shape output) (at 176.53 67.31 0) (fields_autoplaced)
+    (effects (font (size 1.27 1.27)) (justify left))
+  )
   (hierarchical_label "I2C{SCL,SDA}" (shape bidirectional) (at 50.8 43.18 180) (fields_autoplaced)
     (effects (font (size 1.27 1.27)) (justify right))
@@
   (hierarchical_label "INT_EXPANDER" (shape output) (at 50.8 64.77 180) (fields_autoplaced)
     (effects (font (size 1.27 1.27)) (justify right))
+  )
+  (hierarchical_label "MerusChipSelect" (shape output) (at 176.53 64.77 0) (fields_autoplaced)
+    (effects (font (size 1.27 1.27)) (justify left))
   )
   (symbol (lib_id "Device:RotaryEncoder_Switch") (at 260.35 113.03 0) (unit 1)
@@
     )
   )
+  (symbol (lib_id "Connector_Generic:Conn_01x01") (at 149.86 64.77 0) (unit 1)
+    (in_bom yes) (on_board yes) (dnp no) (fields_autoplaced)
+    (property "Reference" "J5" (at 152.4 64.135 0)
+      (effects (font (size 1.27 1.27)) (justify left))
+    )
+    (property "Value" "GPIOB" (at 152.4 66.675 0)
+      (effects (font (size 1.27 1.27)) (justify left))
+    )
+    (property "Footprint" "Connector_PinHeader_2.54mm:PinHeader_1x01_P2.54mm_Vertical" (at 149.86 64.77 0)
+      (effects (font (size 1.27 1.27)) hide)
+    )
+    (property "Datasheet" "~" (at 149.86 64.77 0)
+      (effects (font (size 1.27 1.27)) hide)
+    )
+    (pin "1")
+    (instances
+      (project "esp_radio"
+        (path "/c9e2e0d2-0655-4f5e-8e13-71b41b1f7cfe/6c8b235f-e3ea-4277-bdf9-de9910b169f3"
+          (reference "J5") (unit 1)
+        )
+      )
+    )
+  )
   (symbol (lib_id "Device:R") (at 97.79 87.63 90) (unit 1)
     (in_bom yes) (on_board yes) (dnp no)
@@
         )
       )
-    )
-  )
-  (symbol (lib_id "Connector_Generic:Conn_01x03") (at 149.86 62.23 0) (unit 1)
-    (in_bom yes) (on_board yes) (dnp no) (fields_autoplaced)
-    (property "Reference" "J5" (at 152.4 61.595 0)
-      (effects (font (size 1.27 1.27)) (justify left))
-    )
-    (property "Value" "GPIOB" (at 152.4 64.135 0)
-      (effects (font (size 1.27 1.27)) (justify left))
-    )
-    (property "Footprint" "Connector_PinHeader_2.54mm:PinHeader_1x03_P2.54mm_Vertical" (at 149.86 62.23 0)
-      (effects (font (size 1.27 1.27)) hide)
-    )
-    (property "Datasheet" "~" (at 149.86 62.23 0)
-      (effects (font (size 1.27 1.27)) hide)
-    )
-    (pin "1")
-    (pin "2")
-    (pin "3")
-    (instances
-      (project "esp_radio"
-        (path "/c9e2e0d2-0655-4f5e-8e13-71b41b1f7cfe/6c8b235f-e3ea-4277-bdf9-de9910b169f3"
-          (reference "J5") (unit 1)
-        )
-      )
